File: pcb/environment-monitor.sch (KiCad schematic (older format))
At the start: 14 parts, among them P1 BME280, P2 HEADER, P3 SERIAL, P4 PWR, SW1 RESET, SW2 FLASH, U1 ESP-12E, U2 MCP1700T-3302E/TT

Commit message: Update Schematic and PCB to new design
Parts:
- removed C2: 10uF, Capacitors_SMD:C_1206_HandSoldering, symbol CPOL
- removed P2: HEADER, Pin_Headers:Pin_Header_Straight_1x02, symbol CONN_01X02
- removed P3: SERIAL, Pin_Headers:Pin_Header_Straight_1x06, symbol CONN_01X06
- removed R1: 10R, Resistors_SMD:R_1206_HandSoldering, symbol R
- removed R3: 10k, Resistors_SMD:R_1206_HandSoldering, symbol R
- added C3: 1uF, Capacitors_SMD:C_1206_HandSoldering, symbol C
- added P2: SERIAL, Pin_Headers:Pin_Header_Straight_1x05_Pitch2.54mm, symbol CONN_01X05
- added R4, R5: 4.7k, Resistors_SMD:R_1206_HandSoldering, symbol R
- added SW3: Switch_SPDT_x2, switches:SW_SPDT_PCM12, symbol Switch_SPDT_x2
- C2: renamed from C1; value 1uF -> 10uF
- R1: renamed from R2; value 10k -> 4.7k
- R3: renamed from R6; value 10k -> 4.7k
- U1: value ESP-12E -> ESP-12F
- U2: value MCP1700T-3302E/TT -> MCP1700T; footprint TO_SOT_Packages_SMD:SOT-23_Handsoldering -> smd-semi:SOT-23
- renumbered P4 to P3
Connections:
- net labels added: CH_EN, PWRGND
- wire segments 45 -> 53
- no-connect marks 15 -> 12
Other:
- moved on the sheet: C2, P1, P3, R1, R3, SW1, SW2, U1, U2
